File: kian/kian nest microcontroler/microcontroler.kicad_sch (KiCad schematic)
At the start: 13 parts, among them J1 Conn_01x20_Pin, J2 Conn_01x20_Pin, J4 Conn_01x20_Socket, J5 Conn_01x20_Socket, Q1 NMOS, SW1 SW_MEC_5E, U1 PICO_W, U3 MCP9700x-HLT, U4 MCP9700x-HLT, U5 MCP9700x-HLT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

Commit message: resever
resever is finished
Other:
- moved on the sheet: SW1, U6
Changed lines of the file:
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@@
     (title "microcontroler ")
   )
-  (junction (at 257.81 124.46) (diameter 0) (color 0 0 0 0)
-  )
-  (no_connect (at 215.9 123.19))
+  (junction (at 180.34 118.11) (diameter 0) (color 0 0 0 0)
+  )
+  (no_connect (at 138.43 116.84))
   (no_connect (at 88.9 55.88))
   (wire (pts (xy 208.28 87.63) (xy 214.63 87.63))
@@
     (stroke (width 0) (type default))
   )
-  (wire (pts (xy 257.81 121.92) (xy 257.81 124.46))
+  (wire (pts (xy 180.34 115.57) (xy 180.34 118.11))
     (stroke (width 0) (type default))
   )
@@
     (fill (type none))
   )
-  (rectangle (start 237.49 109.22) (end 261.62 130.81)
+  (rectangle (start 160.02 102.87) (end 184.15 124.46)
     (stroke (width 0) (type default))
     (fill (type none))
   )
-  (rectangle (start 203.2 109.22) (end 234.95 127)
+  (rectangle (start 125.73 102.87) (end 157.48 120.65)
     (stroke (width 0) (type default))
     (fill (type none))
@@
     (effects (font (size 1.27 1.27)) (justify left bottom))
   )
-  (text "reset microcontroler" (at 238.76 111.76 0)
+  (text "reset microcontroler" (at 161.29 105.41 0)
     (effects (font (size 1.27 1.27)) (justify left bottom))
   )
@@
     (effects (font (size 1.27 1.27)) (justify left bottom))
   )
-  (text "safty DTH" (at 204.47 111.76 0)
+  (text "safty DTH" (at 127 105.41 0)
     (effects (font (size 1.27 1.27)) (justify left bottom))
   )
@@
     (effects (font (size 1.27 1.27)) (justify left bottom))
   )
-  (label "run" (at 247.65 124.46 180) (fields_autoplaced)
+  (label "run" (at 170.18 118.11 180) (fields_autoplaced)
     (effects (font (size 1.27 1.27)) (justify right bottom))
   )
-  (label "3.3V pi" (at 215.9 115.57 180) (fields_autoplaced)
+  (label "3.3V pi" (at 138.43 109.22 180) (fields_autoplaced)
     (effects (font (size 1.27 1.27)) (justify right bottom))
   )
@@
     (effects (font (size 1.27 1.27)) (justify left bottom))
   )
-  (label "run" (at 247.65 121.92 180) (fields_autoplaced)
+  (label "run" (at 170.18 115.57 180) (fields_autoplaced)
     (effects (font (size 1.27 1.27)) (justify right bottom))
   )
-  (label "SDA DHT22" (at 215.9 118.11 180) (fields_autoplaced)
+  (label "SDA DHT22" (at 138.43 111.76 180) (fields_autoplaced)
     (effects (font (size 1.27 1.27)) (justify right bottom))
   )
@@
     )
   )
-  (symbol (lib_id "power:GND") (at 215.9 120.65 270) (unit 1)
-    (in_bom yes) (on_board yes) (dnp no) (fields_autoplaced)
-    (property "Reference" "#PWR019" (at 209.55 120.65 0)
-      (effects (font (size 1.27 1.27)) hide)
-    )
-    (property "Value" "GND" (at 212.09 120.65 90)
-      (effects (font (size 1.27 1.27)) (justify right))
-    )
-    (property "Footprint" "" (at 215.9 120.65 0)
-      (effects (font (size 1.27 1.27)) hide)
-    )
-    (property "Datasheet" "" (at 215.9 120.65 0)
+  (symbol (lib_id "power:GND") (at 138.43 114.3 270) (unit 1)
+    (in_bom yes) (on_board yes) (dnp no) (fields_autoplaced)
+    (property "Reference" "#PWR019" (at 132.08 114.3 0)
+      (effects (font (size 1.27 1.27)) hide)
+    )
+    (property "Value" "GND" (at 134.62 114.3 90)
+      (effects (font (size 1.27 1.27)) (justify right))
+    )
+    (property "Footprint" "" (at 138.43 114.3 0)
+      (effects (font (size 1.27 1.27)) hide)
+    )
+    (property "Datasheet" "" (at 138.43 114.3 0)
       (effects (font (size 1.27 1.27)) hide)
     )
@@
     )
   )
-  (symbol (lib_id "power:GND") (at 257.81 124.46 0) (unit 1)
-    (in_bom yes) (on_board yes) (dnp no) (fields_autoplaced)
-    (property "Reference" "#PWR018" (at 257.81 130.81 0)
-      (effects (font (size 1.27 1.27)) hide)
-    )
-    (property "Value" "GND" (at 257.81 129.54 0)
-      (effects (font (size 1.27 1.27)))
-    )
-    (property "Footprint" "" (at 257.81 124.46 0)
-      (effects (font (size 1.27 1.27)) hide)
-    )
-    (property "Datasheet" "" (at 257.81 124.46 0)
+  (symbol (lib_id "power:GND") (at 180.34 118.11 0) (unit 1)
+    (in_bom yes) (on_board yes) (dnp no) (fields_autoplaced)
+    (property "Reference" "#PWR018" (at 180.34 124.46 0)
+      (effects (font (size 1.27 1.27)) hide)
+    )
+    (property "Value" "GND" (at 180.34 123.19 0)
+      (effects (font (size 1.27 1.27)))
+    )
+    (property "Footprint" "" (at 180.34 118.11 0)
+      (effects (font (size 1.27 1.27)) hide)
+    )
+    (property "Datasheet" "" (at 180.34 118.11 0)
       (effects (font (size 1.27 1.27)) hide)
     )
@@
     )
   )
-  (symbol (lib_id "Switch:SW_MEC_5E") (at 252.73 124.46 0) (unit 1)
-    (in_bom yes) (on_board yes) (dnp no) (fields_autoplaced)
-    (property "Reference" "SW1" (at 252.73 114.3 0)
-      (effects (font (size 1.27 1.27)))
-    )
-    (property "Value" "SW_MEC_5E" (at 252.73 116.84 0)
-      (effects (font (size 1.27 1.27)))
-    )
-    (property "Footprint" "" (at 252.73 116.84 0)
-      (effects (font (size 1.27 1.27)) hide)
-    )
-    (property "Datasheet" "http://www.apem.com/int/index.php?controller=attachment&id_attachment=1371" (at 252.73 116.84 0)
-      (effects (font (size 1.27 1.27)) hide)
-    )
-    (property "cost" "2" (at 252.73 124.46 0)
-      (effects (font (size 1.27 1.27)) hide)
-    )
-    (property "where" "brendon" (at 252.73 124.46 0)
+  (symbol (lib_id "Switch:SW_MEC_5E") (at 175.26 118.11 0) (unit 1)
+    (in_bom yes) (on_board yes) (dnp no) (fields_autoplaced)
+    (property "Reference" "SW1" (at 175.26 107.95 0)
+      (effects (font (size 1.27 1.27)))
+    )
+    (property "Value" "SW_MEC_5E" (at 175.26 110.49 0)
+      (effects (font (size 1.27 1.27)))
+    )
+    (property "Footprint" "" (at 175.26 110.49 0)
+      (effects (font (size 1.27 1.27)) hide)
+    )
+    (property "Datasheet" "http://www.apem.com/int/index.php?controller=attachment&id_attachment=1371" (at 175.26 110.49 0)
+      (effects (font (size 1.27 1.27)) hide)
+    )
+    (property "cost" "2" (at 175.26 118.11 0)
+      (effects (font (size 1.27 1.27)) hide)
+    )
+    (property "where" "brendon" (at 175.26 118.11 0)
       (effects (font (size 1.27 1.27)) hide)
     )
@@
     )
   )
-  (symbol (lib_id "partkian:DHT22") (at 222.25 119.38 0) (unit 1)
-    (in_bom yes) (on_board yes) (dnp no) (fields_autoplaced)
-    (property "Reference" "U6" (at 227.33 118.11 0)
+  (symbol (lib_id "partkian:DHT22") (at 144.78 113.03 0) (unit 1)
+    (in_bom yes) (on_board yes) (dnp no) (fields_autoplaced)
+    (property "Reference" "U6" (at 149.86 111.76 0)
       (effects (font (size 1.27 1.27)) (justify left))
     )
-    (property "Value" "DHT22" (at 227.33 120.65 0)
+    (property "Value" "DHT22" (at 149.86 114.3 0)
       (effects (font (size 1.27 1.27)) (justify left))
     )
-    (property "Footprint" "footprint:SENSOR-TH_HAIGU_DHT22" (at 222.25 129.54 0)
+    (property "Footprint" "footprint:SENSOR-TH_HAIGU_DHT22" (at 144.78 123.19 0)
       (effects (font (size 1.27 1.27) italic) hide)
     )
-    (property "Datasheet" "" (at 199.39 110.49 0)
+    (property "Datasheet" "" (at 121.92 104.14 0)
       (effects (font (size 1.27 1.27)) (justify left) hide)
     )
-    (property "LCSC" "C2880291" (at 222.25 110.49 0)
-      (effects (font (size 1.27 1.27)) hide)
-    )
-    (property "where" "https://www.communica.co.za/products/hkd-temp-humd-dht22-sensor?utm_source=www.communica.co.za&variant=44293598052652&sfdr_ptcid=31591_617_694884796&sfdr_hash=9840d3925fc7e58daa080f8556935672&gad_source=1&gclid=CjwKCAjw8diwBhAbEiwA7i_sJVjBvaaYyN6XP6FA_WGJb8ruE_zh2lzVDzIz94sgFtDFTqhCu8xVvRoCdtQQAvD_BwE" (at 222.25 119.38 0)
-      (effects (font (size 1.27 1.27)) hide)
-    )
-    (property "cost" "79" (at 222.25 119.38 0)
-      (effects (font (size 1.27 1.27)) hide)
-    )
+    (property "LCSC" "C2880291" (at 144.78 104.14 0)
+      (effects (font (size 1.27 1.27)) hide)
+    )
+    (property "where" "https://www.communica.co.za/products/hkd-temp-humd-dht22-sensor?utm_source=www.communica.co.za&variant=44293598052652&sfdr_ptcid=31591_617_694884796&sfdr_hash=9840d3925fc7e58daa080f8556935672&gad_source=1&gclid=CjwKCAjw8diwBhAbEiwA7i_sJVjBvaaYyN6XP6FA_WGJb8ruE_zh2lzVDzIz94sgFtDFTqhCu8xVvRoCdtQQAvD_BwE" (at 144.78 113.03 0)
+      (effects (font (size 1.27 1.27)) hide)
+    )
+    (property "cost" "79" (at 144.78 113.03 0)
+      (effects (font (size 1.27 1.27)) hide)
+    )
