File: kian/kian recever microcontroler subsection/microcontroler.kicad_sch (KiCad schematic)
At the start: 2 parts, among them U1 PICO_W

Commit message: resever
resever is finished
Parts:
- removed SD1: ~, symbol pico:SD_card
- added J1, J2: Conn_01x20_Pin, symbol Connector:Conn_01x20_Pin
- added J4, J5: Conn_01x20_Socket, symbol Connector:Conn_01x20_Socket
- added Q1: NMOS, symbol Simulation_SPICE:NMOS
- added SW1: SW_MEC_5E, symbol Switch:SW_MEC_5E
- added U1: ~, symbol partkian:LCD_16X2_LCD_with_I2C_Interface
- added e: ~, symbol partkian:sd_card_reader
- U1: cost (none) -> 150; where (none) -> https://www.pishop.co.za/store/raspberry-pi-pico-wh-with-pr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
Connections:
- net GND: now also Q1.3 (S), SW1.3 (K), SW1.4 (A), U1. (Vcc), e. (SCK); no longer U1.33 (GND_AGND)
- net at U1.16 (GP12_SPI1RX_I2C0SDA_UART0TX): now also U1. (Vcc)
- net at U1.17 (GP13_SPI1CSn_I2C0SCL_UART0RX): now also U1. (Vcc)
- net at U1.2 (GP1_SPI0CSn_I2C0SCL_UART0RX): now also e. (SCK)
- net at U1.29 (GP22): now also Q1.2 (G)
- net run: now reaches U1.30 (RUN)
- net run: now also SW1.1, SW1.2
- net 3.3V pi: now reaches U1.36 (3V3(OUT))
- net 3.3V pi: now also U1. (Vcc), e. (SCK)
- net at U1.37 (3V3_EN): now also Q1.1 (D)
- net at U1.4 (GP2_SPI0SCK_I2C1SDA): now also e. (SCK)
- net at U1.5 (GP3_SPI0TX_I2C1SCL): now also e. (SCK)
- net at U1.6 (GP4_SPI0RX_I2C0SDA_UART1TX): now also e. (SCK)
- net 5V renamed +5V
- new net GNDA: U1.33 (GND_AGND)
- no-connect marks 0 -> 1
Other:
- note added: "SD Card"
- note added: "header for microcontroler"
- note added: "reset microcontroler"
